File: ESP8266_schematic.sch (EAGLE design)
At the start: 32 parts, among them J1 DNP, Q1 600mA/40V, Q2 600mA/40V, U1 ESP8266, U3 W25Q32FV, U4 AP2112K-3.3V, Y1 26MHz

Commit message: Add files via upload
Parts:
- added R7, R9: 10K, rcl:R-US_R0805
Connections:
- net GPIO0: now also R7.2
- net GPIO2/SDA: now also R9.2
- net VCC: now also R7.1, R9.1
Other:
- note added: "ESP8266_CPU"
- note added: "LDO"
- note added: "Programmer_pins"
- note removed: "Voltage Regulator & LiPo Charger"
- moved on the sheet: Q1, Q2, R2, R4
