File: esp8285.sch (EAGLE design)
At the start: 30 parts, among them IC1 ESP8285, Q1 600mA/40V, Q2 600mA/40V, U4 AP2112K-3.3V, Y1 CRYSTAL-26MHZSMD-3.2X2.5

Commit message: Add files via upload
Parts:
- C1: value (none) -> 10uF
- C2: value (none) -> 0.1uF
- L1: value (none) -> DNP
Changed lines of the file:
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@@
 <part name="P+3" library="supply1" library_urn="urn:adsk.eagle:library:371" deviceset="VCC" device=""/>
 <part name="P+4" library="supply1" library_urn="urn:adsk.eagle:library:371" deviceset="VCC" device=""/>
-<part name="L1" library="rcl-2" deviceset="L-US" device="L0603"/>
-<part name="C1" library="rcl" library_urn="urn:adsk.eagle:library:334" deviceset="C-EU" device="C0603" package3d_urn="urn:adsk.eagle:package:23616/2"/>
-<part name="C2" library="rcl" library_urn="urn:adsk.eagle:library:334" deviceset="C-EU" device="C0603" package3d_urn="urn:adsk.eagle:package:23616/2"/>
+<part name="L1" library="rcl-2" deviceset="L-US" device="L0603" value="DNP"/>
+<part name="C1" library="rcl" library_urn="urn:adsk.eagle:library:334" deviceset="C-EU" device="C0603" package3d_urn="urn:adsk.eagle:package:23616/2" value="10uF"/>
+<part name="C2" library="rcl" library_urn="urn:adsk.eagle:library:334" deviceset="C-EU" device="C0603" package3d_urn="urn:adsk.eagle:package:23616/2" value="0.1uF"/>
 <part name="GND1" library="supply1" library_urn="urn:adsk.eagle:library:371" deviceset="GND" device=""/>
 <part name="C3" library="rcl" library_urn="urn:adsk.eagle:library:334" deviceset="C-EU" device="C0603" package3d_urn="urn:adsk.eagle:package:23616/2" value="10uF"/>
@@
 <pinref part="IC1" gate="G$1" pin="EXT_RSTB"/>
 <wire x1="45.72" y1="81.28" x2="45.72" y2="86.36" width="0.1524" layer="91"/>
-<label x="45.72" y="86.36" size="1.778" layer="95" rot="R90" xref="yes"/>
+<label x="45.72" y="86.36" size="0.8128" layer="95" rot="R90" xref="yes"/>
 </segment>
 <segment>
@@
 <pinref part="IC1" gate="G$1" pin="GPIO2"/>
 <wire x1="55.88" y1="22.86" x2="55.88" y2="17.78" width="0.1524" layer="91"/>
-<label x="55.88" y="17.78" size="1.778" layer="95" rot="R270" xref="yes"/>
+<label x="55.88" y="17.78" size="1.016" layer="95" rot="R270" xref="yes"/>
 </segment>
 <segment>
@@
 <pinref part="IC1" gate="G$1" pin="SD_DATA_2"/>
 <wire x1="73.66" y1="45.72" x2="78.74" y2="45.72" width="0.1524" layer="91"/>
-<label x="78.74" y="45.72" size="1.778" layer="95" xref="yes"/>
+<label x="78.74" y="45.72" size="1.016" layer="95" xref="yes"/>
 </segment>
 </net>
@@
 <pinref part="IC1" gate="G$1" pin="SD_DATA_3"/>
 <wire x1="73.66" y1="48.26" x2="78.74" y2="48.26" width="0.1524" layer="91"/>
-<label x="78.74" y="48.26" size="1.778" layer="95" xref="yes"/>
+<label x="78.74" y="48.26" size="1.016" layer="95" xref="yes"/>
 </segment>
 </net>
@@
 <pinref part="IC1" gate="G$1" pin="SD_CMD"/>
 <wire x1="73.66" y1="50.8" x2="78.74" y2="50.8" width="0.1524" layer="91"/>
-<label x="78.74" y="50.8" size="1.778" layer="95" xref="yes"/>
+<label x="78.74" y="50.8" size="1.016" layer="95" xref="yes"/>
 </segment>
 </net>
@@
 <pinref part="IC1" gate="G$1" pin="SD_CLK"/>
 <wire x1="73.66" y1="53.34" x2="78.74" y2="53.34" width="0.1524" layer="91"/>
-<label x="78.74" y="53.34" size="1.778" layer="95" xref="yes"/>
+<label x="78.74" y="53.34" size="1.016" layer="95" xref="yes"/>
 </segment>
 </net>
@@
 <pinref part="IC1" gate="G$1" pin="SD_DATA_0"/>
 <wire x1="73.66" y1="55.88" x2="78.74" y2="55.88" width="0.1524" layer="91"/>
-<label x="78.74" y="55.88" size="1.778" layer="95" xref="yes"/>
+<label x="78.74" y="55.88" size="1.016" layer="95" xref="yes"/>
 </segment>
 </net>
@@
 <pinref part="IC1" gate="G$1" pin="SD_DATA_1"/>
 <wire x1="73.66" y1="58.42" x2="81.28" y2="58.42" width="0.1524" layer="91"/>
-<label x="81.28" y="58.42" size="1.778" layer="95" xref="yes"/>
+<label x="81.28" y="58.42" size="1.016" layer="95" xref="yes"/>
 </segment>
 </net>
@@
 <pinref part="IC1" gate="G$1" pin="GPIO5"/>
 <wire x1="73.66" y1="60.96" x2="78.74" y2="60.96" width="0.1524" layer="91"/>
-<label x="78.74" y="60.96" size="1.778" layer="95" xref="yes"/>
+<label x="78.74" y="60.96" size="1.016" layer="95" xref="yes"/>
 </segment>
 </net>
@@
 <wire x1="63.5" y1="81.28" x2="66.04" y2="81.28" width="0.1524" layer="91"/>
 <wire x1="66.04" y1="81.28" x2="66.04" y2="86.36" width="0.1524" layer="91"/>
-<label x="66.04" y="86.36" size="1.778" layer="95" rot="R90" xref="yes"/>
+<label x="66.04" y="86.36" size="1.016" layer="95" rot="R90" xref="yes"/>
 </segment>
 <segment>
@@
 <wire x1="60.96" y1="83.82" x2="63.5" y2="83.82" width="0.1524" layer="91"/>
 <wire x1="63.5" y1="83.82" x2="63.5" y2="86.36" width="0.1524" layer="91"/>
-<label x="63.5" y="86.36" size="1.778" layer="95" rot="R90" xref="yes"/>
+<label x="63.5" y="86.36" size="1.016" layer="95" rot="R90" xref="yes"/>
 </segment>
 <segment>
@@
 <pinref part="IC1" gate="G$1" pin="RES12K"/>
 <wire x1="48.26" y1="81.28" x2="48.26" y2="86.36" width="0.1524" layer="91"/>
-<label x="48.26" y="86.36" size="1.778" layer="95" rot="R90" xref="yes"/>
-</segment>
-<segment>
+<label x="48.26" y="86.36" size="1.016" layer="95" rot="R90" xref="yes"/>
+</segment>
+<segment>
